Commit message: started implementing the auto pilot and working on tuning the rewards for the model
Took 43 hours 54 minutes

File: simulation/robot.urdf (robot description, URDF)
Before this commit: robot my_robot, 6 links, 5 joints
Joints:
- joint base_to_lidar: origin xyz=0 0 0.3 -> xyz=0 0 0.3 rpy=0 0 3.14159

Commit message: working autopilot
Took 11 hours 43 minutes

File: simulation/robot.urdf (robot description, URDF)
Before this commit: robot my_robot, 6 links, 5 joints
Joints:
- joint base_to_lidar: origin xyz=0 0 0.3 rpy=0 0 3.14159 -> xyz=0 0 0.3 rpy=0 0 0
