Commit message: updated urdf with estimated build positions
Took 1 hour 15 minutes

File: ros2_ws/src/lwf_robot/robot_description/urdf/robot.xacro (robot description, xacro)
@@ -1,199 +1,263 @@
-<?xml version="1.0" ?>
-<robot name="lwf5000" xmlns:xacro="http://www.ros.org/wiki/xacro">
-    <xacro:include filename="$(find robot_description)/urdf/materials.xacro"/>
-    <xacro:include filename="$(find robot_description)/urdf/robot.trans"/>
-    <xacro:include filename="$(find robot_description)/urdf/robot.gazebo"/>
-    <link name="base_link">
-        <inertial>
-            <origin xyz="-0.21590000000000004 0.0 0.10159999999999998" rpy="0 0 0"/>
-            <mass value="209.9379543168"/>
-            <inertia ixx="2.347689" iyy="3.984298" izz="4.887256" ixy="-0.0" iyz="0.0" ixz="-0.0"/>
-        </inertial>
-        <visual>
-            <origin xyz="0 0 0" rpy="0 0 0"/>
-            <geometry>
-                <mesh filename="file://$(find robot_description)/meshes/base_link.stl" scale="0.001 0.001 0.001"/>
-            </geometry>
-            <material name="silver"/>
-        </visual>
-        <collision>
-            <origin xyz="0 0 0" rpy="0 0 0"/>
-            <geometry>
-                <mesh filename="file://$(find robot_description)/meshes/base_link.stl" scale="0.001 0.001 0.001"/>
-            </geometry>
-        </collision>
-    </link>
-    <joint name="base_joint" type="fixed">
-        <parent link="world"/>
-        <child link="base_link"/>
-    </joint>
-    <link name="wheel_front_left_1">
-        <inertial>
-            <origin xyz="1.261521684088318e-17 0.014500000000000013 3.552713678800501e-17" rpy="0 0 0"/>
-            <mass value="3.7075116143850897"/>
-            <inertia ixx="0.005065" iyy="0.00961" izz="0.005065" ixy="-0.0" iyz="-0.0" ixz="0.0"/>
-        </inertial>
-        <visual>
-            <origin xyz="0.0 -0.1524 -0.0" rpy="0 0 0"/>
-            <geometry>
-                <mesh filename="file://$(find robot_description)/meshes/wheel_front_left_1.stl"
-                      scale="0.001 0.001 0.001"/>
-            </geometry>
-            <material name="silver"/>
-        </visual>
-        <collision>
-            <origin xyz="0.0 -0.1524 -0.0" rpy="0 0 0"/>
-            <geometry>
-                <mesh filename="file://$(find robot_description)/meshes/wheel_front_left_1.stl"
-                      scale="0.001 0.001 0.001"/>
-            </geometry>
-        </collision>
-    </link>
-    <link name="wheel_front_right_1">
-        <inertial>
-            <origin xyz="2.101981966549921e-17 -0.015500000000000042 0.006999999999999922" rpy="0 0 0"/>
-            <mass value="3.707511614385092"/>
-            <inertia ixx="0.005065" iyy="0.00961" izz="0.005065" ixy="0.0" iyz="0.0" ixz="-0.0"/>
-        </inertial>
-        <visual>
-            <origin xyz="0.0 0.1524 -0.0" rpy="0 0 0"/>
-            <geometry>
-                <mesh filename="file://$(find robot_description)/meshes/wheel_front_right_1.stl"
-                      scale="0.001 0.001 0.001"/>
-            </geometry>
-            <material name="silver"/>
-        </visual>
-        <collision>
-            <origin xyz="0.0 0.1524 -0.0" rpy="0 0 0"/>
-            <geometry>
-                <mesh filename="file://$(find robot_description)/meshes/wheel_front_right_1.stl"
-                      scale="0.001 0.001 0.001"/>
-            </geometry>
-        </collision>
-    </link>
-    <link name="wheel_rear_right_1">
-        <inertial>
-            <origin xyz="0.0 -0.013499999999999984 -0.002999999999999936" rpy="0 0 0"/>
-            <mass value="3.7075116143850924"/>
-            <inertia ixx="0.005065" iyy="0.00961" izz="0.005065" ixy="-0.0" iyz="-0.0" ixz="0.0"/>
-        </inertial>
-        <visual>
-            <origin xyz="0.4318 0.1524 -0.0" rpy="0 0 0"/>
-            <geometry>
-                <mesh filename="file://$(find robot_description)/meshes/wheel_rear_right_1.stl"
-                      scale="0.001 0.001 0.001"/>
-            </geometry>
-            <material name="silver"/>
-        </visual>
-        <collision>
-            <origin xyz="0.4318 0.1524 -0.0" rpy="0 0 0"/>
-            <geometry>
-                <mesh filename="file://$(find robot_description)/meshes/wheel_rear_right_1.stl"
-                      scale="0.001 0.001 0.001"/>
-            </geometry>
-        </collision>
-    </link>
-    <link name="wheel_rear_left_1">
-        <inertial>
-            <origin xyz="0.0 0.013500000000000095 0.006999999999999993" rpy="0 0 0"/>
-            <mass value="3.707511614385086"/>
-            <inertia ixx="0.005065" iyy="0.00961" izz="0.005065" ixy="-0.0" iyz="-0.0" ixz="0.0"/>
-        </inertial>
-        <visual>
-            <origin xyz="0.4318 -0.1524 -0.0" rpy="0 0 0"/>
-            <geometry>
-                <mesh filename="file://$(find robot_description)/meshes/wheel_rear_left_1.stl"
-                      scale="0.001 0.001 0.001"/>
-            </geometry>
-            <material name="silver"/>
-        </visual>
-        <collision>
-            <origin xyz="0.4318 -0.1524 -0.0" rpy="0 0 0"/>
-            <geometry>
-                <mesh filename="file://$(find robot_description)/meshes/wheel_rear_left_1.stl"
-                      scale="0.001 0.001 0.001"/>
-            </geometry>
-        </collision>
-    </link>
-    <joint name="Rigid 11" type="fixed">
-        <origin xyz="0.0 0.1524 0.0" rpy="0 0 0"/>
-        <parent link="base_link"/>
-        <child link="wheel_front_left_1"/>
-    </joint>
-    <joint name="Revolute 12" type="continuous">
-        <origin xyz="0.0 -0.1524 0.0" rpy="0 0 0"/>
-        <parent link="base_link"/>
-        <child link="wheel_front_right_1"/>
-        <axis xyz="-0.0 0.0 1.0"/>
-    </joint>
-    <joint name="Rigid 13" type="fixed">
-        <origin xyz="-0.4318 -0.1524 0.0" rpy="0 0 0"/>
-        <parent link="base_link"/>
-        <child link="wheel_rear_right_1"/>
-    </joint>
-    <joint name="Rigid 14" type="fixed">
-        <origin xyz="-0.4318 0.1524 0.0" rpy="0 0 0"/>
-        <parent link="base_link"/>
-        <child link="wheel_rear_left_1"/>
-    </joint>
-    <link name="imu_link"/>
-    <joint name="imu_joint" type="fixed">
-        <parent link="base_link"/>
-        <child link="imu_link"/>
-        <origin xyz="0 0 0.2" rpy="0 0 0"/>
-    </joint>
-    <link name="lidar_link"/>
-    <joint name="lidar_joint" type="fixed">
-        <parent link="base_link"/>
-        <child link="lidar_link"/>
-        <origin xyz="0.2 0 0.2" rpy="0 0 0"/>
-    </joint>
-    <link name="cam_front_link"/>
-    <joint name="cam_front_joint" type="fixed">
-        <parent link="base_link"/>
-        <child link="cam_front_link"/>
-        <origin xyz="0.2 0 0.1" rpy="0 0 0"/>
-    </joint>
-    <link name="cam_back_link"/>
-    <joint name="cam_back_joint" type="fixed">
-        <parent link="base_link"/>
-        <child link="cam_back_link"/>
-        <origin xyz="-0.2 0 0.1" rpy="0 0 0"/>
-    </joint>
-    <link name="cam_down_link"/>
-    <joint name="cam_down_joint" type="fixed">
-        <parent link="base_link"/>
-        <child link="cam_down_link"/>
-        <origin xyz="0.2 0 0.1" rpy="0 0 0"/>
-    </joint>
-    <link name="sonar_front_link"/>
-    <joint name="sonar_front_joint" type="fixed">
-        <parent link="base_link"/>
-        <child link="sonar_front_link"/>
-        <origin xyz="0.2 0 0.1" rpy="0 0 0"/>
-    </joint>
-    <link name="sonar_back_link"/>
-    <joint name="sonar_back_joint" type="fixed">
-        <parent link="base_link"/>
-        <child link="sonar_back_link"/>
-        <origin xyz="0.2 0 0.1" rpy="0 0 0"/>
-    </joint>
-    <link name="sonar_left_link"/>
-    <joint name="sonar_left_joint" type="fixed">
-        <parent link="base_link"/>
-        <child link="sonar_left_link"/>
-        <origin xyz="0.2 0 0.1" rpy="0 0 0"/>
-    </joint>
-    <link name="sonar_right_link"/>
-    <joint name="sonar_right_joint" type="fixed">
-        <parent link="base_link"/>
-        <child link="sonar_right_link"/>
-        <origin xyz="0.2 0 0.1" rpy="0 0 0"/>
-    </joint>
-    <link name="magnetometer_link"/>
-    <joint name="magnetometer_joint" type="fixed">
-        <parent link="base_link"/>
-        <child link="magnetometer_link"/>
-        <origin xyz="0 0 0" rpy="0 0 0"/>
-    </joint>
+<?xml version="1.0"?>
+<robot name="lwf5000">
+  <!-- Base Link -->
+  <link name="base_link">
+    <visual>
+      <origin xyz="0 0 0.1715" rpy="0 0 0"/> <!-- Half height of 13.5 inches (0.343 m) -->
+      <geometry>
+        <box size="0.483 0.343 0.343"/> <!-- Length: 19", Width: 13.5", Height: 13.5" -->
+      </geometry>
+      <material name="blue"/>
+    </visual>
+    <collision>
+      <origin xyz="0 0 0.1715" rpy="0 0 0"/>
+      <geometry>
+        <box size="0.483 0.343 0.343"/>
+      </geometry>
+    </collision>
+  </link>
+  <!-- Front Right Wheel -->
+  <link name="front_right_wheel">
+    <visual>
+      <origin xyz="0.1524 -0.2286 0.0762" rpy="0 0 0"/> <!-- X, Y, Z in meters -->
+      <geometry>
+        <cylinder radius="0.08255" length="0.05"/> <!-- Diameter is 6.5 inches -->
+      </geometry>
+      <material name="black"/>
+    </visual>
+  </link>
+  <joint name="front_right_wheel_joint" type="continuous">
+    <parent link="base_link"/>
+    <child link="front_right_wheel"/>
+    <origin xyz="0.1524 -0.2286 0.0762" rpy="0 0 0"/>
+    <axis xyz="0 1 0"/>
+  </joint>
+  <!-- Front Left Wheel -->
+  <link name="front_left_wheel">
+    <visual>
+      <origin xyz="0.1524 0.2286 0.0762" rpy="0 0 0"/>
+      <geometry>
+        <cylinder radius="0.08255" length="0.05"/>
+      </geometry>
+      <material name="black"/>
+    </visual>
+  </link>
+  <joint name="front_left_wheel_joint" type="continuous">
+    <parent link="base_link"/>
+    <child link="front_left_wheel"/>
+    <origin xyz="0.1524 0.2286 0.0762" rpy="0 0 0"/>
+    <axis xyz="0 1 0"/>
+  </joint>
+  <!-- Rear Right Wheel -->
+  <link name="rear_right_wheel">
+    <visual>
+      <origin xyz="-0.1524 -0.2286 0.0762" rpy="0 0 0"/>
+      <geometry>
+        <cylinder radius="0.08255" length="0.05"/>
+      </geometry>
+      <material name="black"/>
+    </visual>
+  </link>
+  <joint name="rear_right_wheel_joint" type="continuous">
+    <parent link="base_link"/>
+    <child link="rear_right_wheel"/>
+    <origin xyz="-0.1524 -0.2286 0.0762" rpy="0 0 0"/>
+    <axis xyz="0 1 0"/>
+  </joint>
+  <!-- Rear Left Wheel -->
+  <link name="rear_left_wheel">
+    <visual>
+      <origin xyz="-0.1524 0.2286 0.0762" rpy="0 0 0"/>
+      <geometry>
+        <cylinder radius="0.08255" length="0.05"/>
+      </geometry>
+      <material name="black"/>
+    </visual>
+  </link>
+  <joint name="rear_left_wheel_joint" type="continuous">
+    <parent link="base_link"/>
+    <child link="rear_left_wheel"/>
+    <origin xyz="-0.1524 0.2286 0.0762" rpy="0 0 0"/>
+    <axis xyz="0 1 0"/>
+  </joint>
+  <!-- IMU Sensor -->
+  <link name="imu_link">
+    <visual>
+      <origin xyz="0 0 0.343" rpy="0 0 0"/>
+      <geometry>
+        <box size="0.02 0.02 0.02"/> <!-- Size for IMU -->
+      </geometry>
+      <material name="green"/>
+    </visual>
+  </link>
+  <joint name="imu_joint" type="fixed">
+    <parent link="base_link"/>
+    <child link="imu_link"/>
+    <origin xyz="0 0 0.343" rpy="0 0 0"/>
+  </joint>
+  <!-- Magnetometer 1 -->
+  <link name="magnetometer_1">
+    <visual>
+      <origin xyz="0 0 0.343" rpy="0 0 0"/>
+      <geometry>
+        <box size="0.02 0.02 0.02"/>
+      </geometry>
+      <material name="red"/>
+    </visual>
+  </link>
+  <joint name="magnetometer_1_joint" type="fixed">
+    <parent link="base_link"/>
+    <child link="magnetometer_1"/>
+    <origin xyz="0 0 0.343" rpy="0 0 0"/>
+  </joint>
+  <!-- Magnetometer 2 -->
+  <link name="magnetometer_2">
+    <visual>
+      <origin xyz="-0.0254 -0.1524 0.343" rpy="0 0 0"/>
+      <geometry>
+        <box size="0.02 0.02 0.02"/>
+      </geometry>
+      <material name="red"/>
+    </visual>
+  </link>
+  <joint name="magnetometer_2_joint" type="fixed">
+    <parent link="base_link"/>
+    <child link="magnetometer_2"/>
+    <origin xyz="-0.0254 -0.1524 0.343" rpy="0 0 0"/>
+  </joint>
+  <!-- PTZ Camera -->
+  <link name="ptz_camera_link">
+    <visual>
+      <origin xyz="0.2413 -0.1143 0.419" rpy="0 0 0"/>
+      <geometry>
+        <box size="0.05 0.05 0.1"/> <!-- PTZ camera model -->
+      </geometry>
+      <material name="black"/>
+    </visual>
+  </link>
+  <joint name="ptz_camera_joint" type="fixed">
+    <parent link="base_link"/>
+    <child link="ptz_camera_link"/>
+    <origin xyz="0.2413 -0.1143 0.419" rpy="0 0 0"/>
+  </joint>
+  <!-- Lidar -->
+  <link name="lidar_link">
+    <visual>
+      <origin xyz="0.0254 0.0254 0.4445" rpy="0 0 0"/>
+      <geometry>
+        <cylinder radius="0.05" length="0.1"/> <!-- Simplified lidar -->
+      </geometry>
+      <material name="blue"/>
+    </visual>
+  </link>
+  <joint name="lidar_joint" type="fixed">
+    <parent link="base_link"/>
+    <child link="lidar_link"/>
+    <origin xyz="0.0254 0.0254 0.4445" rpy="0 0 0"/>
+  </joint>
+  <!-- RGB-D Camera -->
+  <link name="rgbd_camera">
+    <visual>
+      <origin xyz="0.2159 0 0.3556" rpy="0 0 0"/> <!-- Front RGB-D Camera -->
+      <geometry>
+        <box size="0.03 0.03 0.05"/> <!-- Simplified depth camera -->
+      </geometry>
+      <material name="blue"/>
+    </visual>
+  </link>
+  <joint name="rgbd_camera_joint" type="fixed">
+    <parent link="base_link"/>
+    <child link="rgbd_camera"/>
+    <origin xyz="0.2159 0 0.3556" rpy="0 0 0"/>
+  </joint>
+  <!-- Front Sonar -->
+  <link name="front_sonar">
+    <visual>
+      <origin xyz="0.2032 0 0.2159" rpy="0 0 0"/>
+      <geometry>
+        <cylinder radius="0.01" length="0.05"/> <!-- Sonar model -->
+      </geometry>
+      <material name="gray"/>
+    </visual>
+  </link>
+  <joint name="front_sonar_joint" type="fixed">
+    <parent link="base_link"/>
+    <child link="front_sonar"/>
+    <origin xyz="0.2032 0 0.2159" rpy="0 0 0"/>
+  </joint>
+  <!-- Right Sonar -->
+  <link name="right_sonar">
+    <visual>
+      <origin xyz="0 -0.17145 0.2159" rpy="0 0 -1.5708"/> <!-- Pointing right -->
+      <geometry>
+        <cylinder radius="0.01" length="0.05"/>
+      </geometry>
+      <material name="gray"/>
+    </visual>
+  </link>
+  <joint name="right_sonar_joint" type="fixed">
+    <parent link="base_link"/>
+    <child link="right_sonar"/>
+    <origin xyz="0 -0.17145 0.2159" rpy="0 0 -1.5708"/>
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