Commit message: stuff
Took 20 minutes

File: ros2_ws/src/lwf_robot/urdf/lwf_robot.urdf (robot description, URDF)
Before this commit: robot lwf5000, 17 links, 16 joints
Joints:
- joint front_left_wheel_joint: origin xyz=0.1524 0.2286 0.0762 rpy=0 0 0 -> xyz=0.1524 0.2286 0.0762 rpy=1.5708 0 0
- joint front_right_wheel_joint: origin xyz=0.1524 -0.2286 0.0762 rpy=0 0 0 -> xyz=0.1524 -0.2286 0.0762 rpy=-1.5708 0 0
- joint rear_left_wheel_joint: origin xyz=-0.1524 0.2286 0.0762 rpy=0 0 0 -> xyz=-0.1524 0.2286 0.0762 rpy=1.5708 0 0
- joint rear_right_wheel_joint: origin xyz=-0.1524 -0.2286 0.0762 rpy=0 0 0 -> xyz=-0.1524 -0.2286 0.0762 rpy=-1.5708 0 0

Commit message: stuff
Took 5 minutes

File: ros2_ws/src/lwf_robot/urdf/lwf_robot.urdf (robot description, URDF)
Before this commit: robot lwf5000, 17 links, 16 joints
Joints:
- joint front_right_wheel_joint: origin xyz=0.1524 -0.2286 0.0762 rpy=-1.5708 0 0 -> xyz=0.1524 -0.2286 0.0762 rpy=0 0 0

Commit message: stuff
Took 7 minutes

File: ros2_ws/src/lwf_robot/urdf/lwf_robot.urdf (robot description, URDF)
Before this commit: robot lwf5000, 17 links, 16 joints
Joints:
- joint front_right_wheel_joint: origin xyz=0.1524 -0.2286 0.0762 rpy=0 0 0 -> xyz=0 0 0 rpy=0 0 0

Commit message: stuff
Took 9 minutes

File: ros2_ws/src/lwf_robot/urdf/lwf_robot.urdf (robot description, URDF)
Before this commit: robot lwf5000, 17 links, 16 joints
Joints:
- joint front_right_wheel_joint: origin xyz=0 0 0 rpy=0 0 0 -> xyz=0.1524 -0.2286 0.0762 rpy=0 0 0

Commit message: stuff
Took 4 minutes

File: ros2_ws/src/lwf_robot/urdf/lwf_robot.urdf (robot description, URDF)
Before this commit: robot lwf5000, 17 links, 16 joints
Joints:
- joint front_right_wheel_joint: origin xyz=0.1524 -0.2286 0.0762 rpy=0 0 0 -> (none)

Commit message: stuff
Took 11 minutes

File: ros2_ws/src/lwf_robot/urdf/lwf_robot.urdf (robot description, URDF)
Before this commit: robot lwf5000, 17 links, 16 joints
Joints:
- joint front_right_wheel_joint: origin (none) -> xyz=0.1524 -0.2286 0.0762 rpy=0 0 0

Commit message: stuff
Took 8 minutes

File: ros2_ws/src/lwf_robot/urdf/lwf_robot.urdf (robot description, URDF)
Before this commit: robot lwf5000, 17 links, 16 joints
Joints:
- joint front_left_wheel_joint: origin xyz=0.1524 0.2286 0.0762 rpy=1.5708 0 0 -> xyz=0.1524 0.17145 0.0762 rpy=1.5708 0 0
- joint front_right_wheel_joint: origin xyz=0.1524 -0.2286 0.0762 rpy=0 0 0 -> xyz=0.1524 -0.17145 0.0762 rpy=0 0 0

Commit message: stuff
Took 13 minutes

File: ros2_ws/src/lwf_robot/urdf/lwf_robot.urdf (robot description, URDF)
Before this commit: robot lwf5000, 17 links, 16 joints
Joints:
- joint front_left_wheel_joint: origin xyz=0.1524 0.17145 0.0762 rpy=1.5708 0 0 -> xyz=0.1524 0.17145 0.0762 rpy=0 0 0

Commit message: stuff
Took 3 minutes

File: ros2_ws/src/lwf_robot/urdf/lwf_robot.urdf (robot description, URDF)
Before this commit: robot lwf5000, 17 links, 16 joints
Joints:
- joint rear_left_wheel_joint: origin xyz=-0.1524 0.2286 0.0762 rpy=1.5708 0 0 -> xyz=-0.1524 0.2286 0.0762 rpy=0 0 0
- joint rear_right_wheel_joint: origin xyz=-0.1524 -0.2286 0.0762 rpy=-1.5708 0 0 -> xyz=-0.1524 -0.2286 0.0762 rpy=0 0 0

Commit message: stuff
Took 3 minutes

File: ros2_ws/src/lwf_robot/urdf/lwf_robot.urdf (robot description, URDF)
Before this commit: robot lwf5000, 17 links, 16 joints
Joints:
- joint rear_left_wheel_joint: origin xyz=-0.1524 0.2286 0.0762 rpy=0 0 0 -> xyz=-0.1524 0.17145 0.0762 rpy=0 0 0
- joint rear_right_wheel_joint: origin xyz=-0.1524 -0.2286 0.0762 rpy=0 0 0 -> xyz=-0.1524 -0.17145 0.0762 rpy=0 0 0

Commit message: stuff
Took 4 minutes

File: ros2_ws/src/lwf_robot/urdf/lwf_robot.urdf (robot description, URDF)
Before this commit: robot lwf5000, 17 links, 16 joints
Joints:
- joint front_camera_joint: origin xyz=0.2159 0.0508 0.3556 rpy=0 0 0 -> xyz=0.2159 0.0508 0.4 rpy=0 0 0
- joint imu_joint: origin xyz=0 0 0.343 rpy=0 0 0 -> xyz=0 0 0.4 rpy=0 0 0
- joint magnetometer_1_joint: origin xyz=0 0 0.343 rpy=0 0 0 -> xyz=0 0 0.4 rpy=0 0 0
- joint magnetometer_2_joint: origin xyz=-0.0254 -0.1524 0.343 rpy=0 0 0 -> xyz=-0.0254 -0.1524 0.4 rpy=0 0 0
- joint rear_camera_joint: origin xyz=-0.2159 -0.0508 0.4064 rpy=0 0 3.14159 -> xyz=-0.2159 -0.0508 0.5 rpy=0 0 3.14159
- joint rgbd_camera_joint: origin xyz=0.2159 0 0.3556 rpy=0 0 0 -> xyz=0.2159 0 0.4 rpy=0 0 0

Commit message: adding inertial entrires for all links
Took 14 minutes

File: ros2_ws/src/lwf_robot/urdf/lwf_robot.urdf (robot description, URDF)
Before this commit: robot lwf5000, 17 links, 16 joints
Links:
- link base_link: mass None -> 8.0
- link front_camera: mass None -> 0.5
- link front_left_wheel: mass None -> 1.25
- link front_right_wheel: mass None -> 1.25
- link front_sonar: mass None -> 0.5
- link imu_link: mass None -> 0.5
- link left_sonar: mass None -> 0.5
- link lidar_link: mass None -> 0.5
- link magnetometer_1: mass None -> 0.5
- link magnetometer_2: mass None -> 0.5
- link ptz_camera_link: mass None -> 0.5
- link rear_camera: mass None -> 0.5
- link rear_left_wheel: mass None -> 1.25
- link rear_right_wheel: mass None -> 1.25
- link rear_sonar: mass None -> 0.5
- link rgbd_camera: mass None -> 0.5
- link right_sonar: mass None -> 0.5

Commit message: changes
Took 10 minutes

File: ros2_ws/src/lwf_robot/urdf/lwf_robot.urdf (robot description, URDF)
Before this commit: robot lwf5000, 17 links, 16 joints
Links:
- added link camera_color_frame, mass 0.5; visual box size=0.03 0.03 0.05
- added link camera_color_optical_frame, mass 0.5; visual box size=0.03 0.03 0.05
- added link camera_depth_frame, mass 0.5; visual box size=0.03 0.03 0.05
- added link camera_depth_optical_frame, mass 0.5; visual box size=0.03 0.03 0.05
- added link camera_link, mass 0.5; visual box size=0.03 0.03 0.05
Joints:
- added joint camera_color_frame_joint: type fixed, parent rgbd_camera, child camera_color_frame, origin xyz=0.2159 0 0.4 rpy=0 0 0
- added joint camera_color_optical_frame_joint: type fixed, parent rgbd_camera, child camera_color_optical_frame, origin xyz=0.2159 0 0.4 rpy=0 0 0
- added joint camera_depth_frame_joint: type fixed, parent rgbd_camera, child camera_depth_frame, origin xyz=0.2159 0 0.4 rpy=0 0 0
- added joint camera_depth_optical_frame_joint: type fixed, parent rgbd_camera, child camera_depth_optical_frame, origin xyz=0.2159 0 0.4 rpy=0 0 0
- added joint camera_link_joint: type fixed, parent rgbd_camera, child camera_link, origin xyz=0.2159 0 0.4 rpy=0 0 0

Commit message: build fix? maybe?
Took 50 minutes

File: ros2_ws/src/lwf_robot/urdf/lwf_robot.urdf (robot description, URDF)
Before this commit: robot lwf5000, 22 links, 21 joints
Links:
- removed link lidar_link
- added link lidar_frame, mass 0.5; visual cylinder length=0.1 radius=0.05

Commit message: build fix? maybe?
Took 37 minutes

File: ros2_ws/src/lwf_robot/urdf/lwf_robot.urdf (robot description, URDF)
Before this commit: robot lwf5000, 22 links, 21 joints
Joints:
- joint lidar_joint: child lidar_link -> lidar_frame

Commit message: build fix? maybe?
Took 13 minutes

File: ros2_ws/src/lwf_robot/urdf/lwf_robot.urdf (robot description, URDF)
Before this commit: robot lwf5000, 22 links, 21 joints
Links:
- removed link lidar_frame
- added link laser_frame, mass 0.5; visual cylinder length=0.1 radius=0.05
Joints:
- joint lidar_joint: child lidar_frame -> laser_frame

Commit message: build fix? maybe?
Took 9 minutes

File: ros2_ws/src/lwf_robot/urdf/lwf_robot.urdf (robot description, URDF)
Before this commit: robot lwf5000, 22 links, 21 joints
Links:
- removed link laser_frame
- added link laser, mass 0.5; visual cylinder length=0.1 radius=0.05
Joints:
- joint lidar_joint: child laser_frame -> laser

Commit message: build fix? maybe?
Took 32 minutes

File: ros2_ws/src/lwf_robot/urdf/lwf_robot.urdf (robot description, URDF)
Before this commit: robot lwf5000, 22 links, 21 joints
Links:
- removed link camera_link
- added link camera, mass 0.5; visual box size=0.03 0.03 0.05
Joints:
- joint camera_color_frame_joint: parent rgbd_camera -> camera
- joint camera_color_optical_frame_joint: parent rgbd_camera -> camera
- joint camera_depth_frame_joint: parent rgbd_camera -> camera
- joint camera_depth_optical_frame_joint: parent rgbd_camera -> camera
- joint camera_link_joint: child camera_link -> camera

Commit message: build fix? maybe?
Took 2 hours 6 minutes

File: ros2_ws/src/lwf_robot/urdf/lwf_robot.urdf (robot description, URDF)
Before this commit: robot lwf5000, 22 links, 21 joints
Links:
- removed link imu_link
- removed link rgbd_camera
- added link camera_imu_frame; visual box size=0.03 0.03 0.05
- added link imu_frame, mass 0.5; visual box size=0.02 0.02 0.02
- added link rgbd_camera_frame, mass 0.5; visual box size=0.03 0.03 0.05
- link camera: mass 0.5 -> None
- link camera_color_optical_frame: mass 0.5 -> None
- link camera_depth_frame: mass 0.5 -> None
- link camera_depth_optical_frame: mass 0.5 -> None
Joints:
- added joint camera_imu_frame_joint: type fixed, parent camera, child camera_imu_frame, origin xyz=0.2159 0 0.4 rpy=0 0 0
- joint camera_depth_optical_frame_joint: parent camera -> camera_depth_frame
- joint camera_link_joint: parent rgbd_camera -> rgbd_camera_frame
- joint imu_joint: child imu_link -> imu_frame
- joint rgbd_camera_joint: child rgbd_camera -> rgbd_camera_frame
